File: source/pcb/comet.kicad_sch (KiCad schematic)
At the start: 76 parts, among them J1 USB_C_Receptacle_USB2.0_14P, J3 Conn_01x12, J4 Conn_01x02, J5 Micro_SD_Card_Det1, SW1 SW_Push, SW10 SW_Push, SW11 SW_SPDT, SW2 SW_Push, SW3 SW_Push, SW4 SW_Push, SW5 SW_Push, SW6 SW_Push, SW7 SW_Push, SW8 SW_Push, SW9 SW_Push, U1 LIS2DH, U2 IP5306, U3 RP2354A, U4 XC6206PxxxMR, U5 MAX98357A, Y1 Crystal_GND24

Commit message: Update JOURNAL.md
Parts:
- added C48: 0.1uF, Capacitor_SMD:C_0402_1005Metric, symbol Device:C_Small
- added C49: 10uF, Capacitor_SMD:C_0402_1005Metric, symbol Device:C_Small
- H5: renamed from H9; footprint MountingHole:MountingHole_3.2mm_M3 -> common_footprints:display_hole
- LS1: footprint (none) -> Connector_PinSocket_2.54mm:PinSocket_1x02_P2.54mm_Vertical
- SW10, SW3, SW4, SW5, SW6, SW7, SW8, SW9: footprint footprints:button_342 -> common_footprints:SW-SMD_6x6
- SW11: footprint (none) -> common_footprints:SW-TH_MSK12D18G2
Connections:
- net +3V3: now also C48.1, C49.1
- net GND: now also C48.2, C49.2
